Commit message: Fix A: Spawn Edited Fix B: Removed the LiDAR plugin Fix C: All namespace prefixes consistent Fix E: Entry points fixed Fix F: Cleaned up unused R200/Astra mesh files

File: ros2_ws/src/robot_description_pkg/robot_description_pkg_fixed/urdf/tb3_custom.urdf.xacro (robot description, xacro)
@@ -1,12 +1,12 @@
 <?xml version="1.0" ?>
 <robot name="turtlebot3_burger" xmlns:xacro="http://ros.org/wiki/xacro">
-  <!--
-    Customised TurtleBot3 Burger URDF (Xacro)
-    Namespace argument supports multi-robot spawning.
-    Usage:  xacro tb3_custom.urdf.xacro namespace:=robot1/
-  -->
+  <!-- ───────────────────────────────────────────────────
+       Namespace argument — supports multi-robot spawning.
+       Usage:  xacro tb3_custom.urdf.xacro namespace:=robot1/
+       Default is empty string (single-robot use).
+  ─────────────────────────────────────────────────────── -->
   <xacro:arg name="namespace" default=""/>
   <xacro:property name="namespace" value="$(arg namespace)"/>
-  <!-- Materials -->
+  <!-- ── Materials ──────────────────────────────────── -->
   <material name="black">      <color rgba="0.0 0.0 0.0 1.0"/></material>
   <material name="dark">       <color rgba="0.3 0.3 0.3 1.0"/></material>
@@ -19,5 +19,5 @@
   <material name="red">        <color rgba="0.8 0.0 0.0 1.0"/></material>
   <material name="white">      <color rgba="1.0 1.0 1.0 1.0"/></material>
-  <!-- Base footprint -->
+  <!-- ── Base footprint (virtual floor-level origin) ── -->
   <link name="${namespace}base_footprint"/>
   <joint name="${namespace}base_joint" type="fixed">
@@ -26,10 +26,11 @@
     <origin xyz="0.0 0.0 0.010" rpy="0 0 0"/>
   </joint>
-  <!-- Base link -->
+  <!-- ── Base link (chassis) ──────────────────────── -->
   <link name="${namespace}base_link">
     <visual>
       <origin xyz="-0.032 0 0.0" rpy="0 0 0"/>
       <geometry>
-        <mesh filename="file://$(find robot_description_pkg)/meshes/bases/burger_base.stl" scale="0.001 0.001 0.001"/>
+        <mesh filename="file://$(find robot_description_pkg)/meshes/bases/burger_base.stl"
+              scale="0.001 0.001 0.001"/>
       </geometry>
       <material name="light_black"/>
@@ -46,5 +47,5 @@
     </inertial>
   </link>
-  <!-- Left wheel -->
+  <!-- ── Left wheel ───────────────────────────────── -->
   <joint name="${namespace}wheel_left_joint" type="continuous">
     <parent link="${namespace}base_link"/>
@@ -57,5 +58,6 @@
       <origin xyz="0 0 0" rpy="1.57 0 0"/>
       <geometry>
-        <mesh filename="file://$(find robot_description_pkg)/meshes/wheels/left_tire.stl" scale="0.001 0.001 0.001"/>
+        <mesh filename="file://$(find robot_description_pkg)/meshes/wheels/left_tire.stl"
+              scale="0.001 0.001 0.001"/>
       </geometry>
       <material name="dark"/>
@@ -72,5 +74,5 @@
     </inertial>
   </link>
-  <!-- Right wheel -->
+  <!-- ── Right wheel ──────────────────────────────── -->
   <joint name="${namespace}wheel_right_joint" type="continuous">
     <parent link="${namespace}base_link"/>
@@ -83,5 +85,6 @@
       <origin xyz="0 0 0" rpy="1.57 0 0"/>
       <geometry>
-        <mesh filename="file://$(find robot_description_pkg)/meshes/wheels/right_tire.stl" scale="0.001 0.001 0.001"/>
+        <mesh filename="file://$(find robot_description_pkg)/meshes/wheels/right_tire.stl"
+              scale="0.001 0.001 0.001"/>
       </geometry>
       <material name="dark"/>
@@ -98,5 +101,5 @@
     </inertial>
   </link>
-  <!-- Rear caster (fixed skid plate) -->
+  <!-- ── Rear caster ──────────────────────────────── -->
   <joint name="${namespace}caster_back_joint" type="fixed">
     <parent link="${namespace}base_link"/>
@@ -116,5 +119,5 @@
     </inertial>
   </link>
-  <!-- IMU -->
+  <!-- ── IMU ──────────────────────────────────────── -->
   <joint name="${namespace}imu_joint" type="fixed">
     <parent link="${namespace}base_link"/>
@@ -123,5 +126,5 @@
   </joint>
   <link name="${namespace}imu_link"/>
-  <!-- LiDAR mount (visual only - no sensor plugin, project does not use LiDAR) -->
+  <!-- ── LiDAR (LDS-01) ───────────────────────────── -->
   <joint name="${namespace}scan_joint" type="fixed">
     <parent link="${namespace}base_link"/>
@@ -133,5 +136,6 @@
       <origin xyz="0 0 0.0" rpy="0 0 0"/>
       <geometry>
-        <mesh filename="file://$(find robot_description_pkg)/meshes/sensors/lds.stl" scale="0.001 0.001 0.001"/>
+        <mesh filename="file://$(find robot_description_pkg)/meshes/sensors/lds.stl"
+              scale="0.001 0.001 0.001"/>
       </geometry>
       <material name="dark"/>
@@ -148,5 +152,9 @@
     </inertial>
   </link>
-  <!-- GPS (now properly namespaced) -->
+  <!-- ── GPS ─────────────────────────────────────────
+       FIX: ${namespace} prefix added to both the link
+       and the joint child so the TF tree is consistent
+       with every other link when a namespace is used.
+  ─────────────────────────────────────────────────── -->
   <link name="${namespace}gps_link">
     <inertial>
@@ -162,61 +170,31 @@
     <origin xyz="0.0 0.0 0.15" rpy="0 0 0"/>
   </joint>
-  <!--
-    ==================================================
-    Contact dynamics  -  the complete anti-drift tuning
-    ==================================================
-    Just setting mu1/mu2 is not enough. Three independent
-    effects need tuning to fully prevent drift:
-    1. STICK-SLIP at the wheels.
-       mu1=2.0 (original) is grippier than real rubber on
-       smooth flooring. ODE then alternates between stick
-       (no slip) and slip (kinetic friction), producing
-       tiny sideways pulses that integrate into drift.
-       mu1=mu2=1.0 stays in the smooth-friction regime.
-    2. CONTACT CHATTER at the caster.
-       The caster collision is a box. Edges and corners
-       enter and leave contact frame-by-frame as the body
-       oscillates by micrometre-scale amounts. kp (contact
-       stiffness) and kd (contact damping) make the contact
-       softly compliant so the box settles instead of
-       bouncing. minDepth lets ODE accept a tiny penetration
-       without applying a corrective velocity. minDepth is
-       the single most important parameter against drift.
-    3. MAX CORRECTING VELOCITY.
-       maxVel caps the corrective velocity ODE applies on
-       a constraint. Without it, a single penetrated frame
-       can launch the body sideways at metres per second for
-       one step - visible drift. 0.1 m/s is conservative.
-    Wheels also get fdir1 (primary friction direction), which
-    locks friction along the rolling direction and prevents
-    ODE from re-deriving the contact frame each step.
-  -->
+  <!-- ── Wheel friction (Gazebo) ──────────────────── -->
   <gazebo reference="${namespace}wheel_left_link">
-    <mu1>1.0</mu1>
-    <mu2>1.0</mu2>
-    <kp>1000000.0</kp>
-    <kd>100.0</kd>
-    <minDepth>0.001</minDepth>
-    <maxVel>0.1</maxVel>
-    <fdir1>1 0 0</fdir1>
+    <mu1>2.0</mu1>
+    <mu2>2.0</mu2>
   </gazebo>
   <gazebo reference="${namespace}wheel_right_link">
-    <mu1>1.0</mu1>
-    <mu2>1.0</mu2>
-    <kp>1000000.0</kp>
-    <kd>100.0</kd>
-    <minDepth>0.001</minDepth>
-    <maxVel>0.1</maxVel>
-    <fdir1>1 0 0</fdir1>
+    <mu1>2.0</mu1>
+    <mu2>2.0</mu2>
   </gazebo>
+  <!-- ── Caster friction (Gazebo) ─────────────────────
+       *** THE DRIFT FIX ***
+       The "caster" in this URDF is a fixed box rigidly
+       attached to base_link — it's a skid plate, NOT a
+       rolling caster wheel.  With Gazebo's default
+       friction (mu ≈ 1.0) the box drags on the floor
+       and creates asymmetric forces that push the
+       robot off its commanded path (visible drift,
+       especially during turns or at rest).
+       Setting mu1 = mu2 = 0 makes the caster frictionless
+       so it slides freely and the wheels alone determine
+       motion. This is the standard TurtleBot3 fix.
+  ─────────────────────────────────────────────────── -->
   <gazebo reference="${namespace}caster_back_link">
     <mu1>0.0</mu1>
     <mu2>0.0</mu2>
-    <kp>1000000.0</kp>
-    <kd>100.0</kd>
-    <minDepth>0.001</minDepth>
-    <maxVel>0.1</maxVel>
   </gazebo>
-  <!-- Sensor and actuator plugins -->
+  <!-- ── Sensor & actuator plugins ────────────────── -->
   <xacro:include filename="$(find robot_description_pkg)/urdf/tb3_sensors.gazebo.xacro"/>
 </robot>

File: ros2_ws/src/robot_description_pkg/robot_description_pkg_fixed/urdf/tb3_sensors.gazebo.xacro (robot description, xacro)
@@ -2,15 +2,25 @@
 <robot xmlns:xacro="http://www.ros.org/wiki/xacro">
   <!--
-    Gazebo sensor and actuator plugins.
-    Included by tb3_custom.urdf.xacro which defines ${namespace}.
-    Sensors:  IMU (libgazebo_ros_imu_sensor.so) -> /imu/data
-              GPS (libgazebo_ros_gps_sensor.so) -> /gps/fix
-    Actuator: differential drive (libgazebo_ros_diff_drive.so)
-              -> /cmd_vel (sub), /odom (pub)
-    There is intentionally NO LiDAR plugin; this project does
-    not use a laser scanner. The base_scan link in the URDF is
-    kept for its visual mesh only.
+    Gazebo sensor & actuator plugins for the customised TurtleBot3 Burger.
+    Included by tb3_custom.urdf.xacro which defines the ${namespace}
+    xacro property, so all link / joint / frame references here use
+    that same prefix.
+    Sensors
+    ======
+    1. IMU        — libgazebo_ros_imu_sensor.so   → /imu/data
+    2. GPS        — libgazebo_ros_gps_sensor.so   → /gps/fix
+    NOTE: The base_scan link in the URDF is kept only for its visual
+    mesh (so the robot still looks correct). There is intentionally
+    NO LiDAR sensor plugin — this project does not use a laser scanner.
+    Actuator
+    ======-
+    3. Diff-drive — libgazebo_ros_diff_drive.so   → /cmd_vel, /odom
   -->
-  <!-- IMU (100 Hz) -->
+  <!-- ═══════════════════════════════════════════════
+       1.  IMU  (BMI160-like — 100 Hz)
+       Now uses ${namespace}imu_link so the TF and
+       gazebo reference stay consistent under any
+       namespace.
+  ═══════════════════════════════════════════════════ -->
   <gazebo reference="${namespace}imu_link">
     <sensor name="tb3_imu" type="imu">
@@ -39,5 +49,8 @@
     </sensor>
   </gazebo>
-  <!-- GPS (5 Hz) -->
+  <!-- ═══════════════════════════════════════════════
+       2.  GPS  (5 Hz, ~0.32 m horizontal stddev)
+       Now uses ${namespace}gps_link.
+  ═══════════════════════════════════════════════════ -->
   <gazebo reference="${namespace}gps_link">
     <sensor name="tb3_gps" type="gps">
@@ -63,5 +76,16 @@
     </sensor>
   </gazebo>
-  <!-- Differential drive (30 Hz) -->
+  <!-- ═══════════════════════════════════════════════
+       3.  Differential Drive  (30 Hz)
+       Fixes vs. original:
+         - left/right joint names use ${namespace} so
+           the plugin finds the joints in any namespace.
+         - robot_base_frame uses ${namespace}.
+         - publish_odom_tf = true so the odom → base_footprint
+           TF is published  and the package works standalone.
+           Switch to false if/when you add an EKF node
+           (e.g. robot_localization) that will own that
+           edge of the TF tree.
+  ═══════════════════════════════════════════════════ -->
   <gazebo>
     <plugin name="tb3_diff_drive" filename="libgazebo_ros_diff_drive.so">
@@ -79,5 +103,5 @@
       <max_wheel_acceleration>1.0</max_wheel_acceleration>
       <publish_odom>true</publish_odom>
-      <publish_odom_tf>true</publish_odom_tf>
+      <publish_odom_tf>true</publish_odom_tf>   <!-- set false when an EKF takes over -->
       <publish_wheel_tf>false</publish_wheel_tf>
       <odometry_frame>odom</odometry_frame>
